Commit message: updating urdf

File: urdf/manipulator.urdf (robot description, URDF)
Before this commit: robot robot_diff, 7 links, 6 joints
Links:
- added link Motor3R, mass 0.16505359; collision mesh filename=package://manipulator_description/meshes/motor3R.dae; visual mesh filename=package://manipulator_description/meshes/motor3R.dae
Joints:
- added joint motor3r_elo2: type fixed, parent Elo2, child Motor3R, origin xyz=0.026 ${0.47211676-0.02086310} -0.036 rpy=0 1.571 0
- joint elo2_motor2: origin xyz=0 -0.03 0 rpy=0 0 0 -> xyz=${0.2275-0.22765252} -0.04 ${-0.067+0.0381+0.02935} rpy=0 0 -1.571

Commit message: change the joint

File: urdf/manipulator.urdf (robot description, URDF)
Before this commit: robot robot_diff, 8 links, 7 joints
Links:
- added link Motor3T, mass 0.16499216; collision mesh filename=package://manipulator_description/meshes/motor3T.dae; visual mesh filename=package://manipulator_description/meshes/motor3T.dae
Joints:
- added joint motor3t_elo2: type fixed, parent Elo2, child Motor3T, origin xyz=-0.026 ${0.47211676-0.02086310} -0.03 rpy=0 -1.571 0
- joint elo2_motor2: limit (none) -> lower=-1.77 upper=1.77 effort=1000.0 velocity=0.5; type continuous -> revolute
- joint motor3r_elo2: origin xyz=0.026 ${0.47211676-0.02086310} -0.036 rpy=0 1.571 0 -> xyz=0.026 ${0.47211676-0.02086310} -0.03 rpy=0 1.571 0
